File: eagle/controller.brd (EAGLE design)
At the start: 70.8 x 21.6 mm, 10 parts, among them IC1 ULN2003AD, IC2 ULN2003AD, K1 68711814022, U1 ARDUINO_PRO_MINI

Commit message: traced the board
Parts:
- moved JP3 2.54 mm to (66.0, 77.5), turned to 90 degrees
Routing:
- net GND: track 0.00 -> 102.3 mm, vias 0 -> 2
- net V+: track 0.00 -> 46.3 mm
- net N$1: track 0.00 -> 43.6 mm
- net N$14: track 0.00 -> 43.1 mm
- net N$15: track 0.00 -> 40.8 mm
- net N$3: track 0.00 -> 40.8 mm
- net N$2: track 0.00 -> 39.5 mm
- net N$30: track 0.00 -> 38.4 mm
- net N$16: track 0.00 -> 36.8 mm
- net N$13: track 0.00 -> 36.4 mm
- net N$19: track 0.00 -> 33.4 mm, vias 0 -> 1
- net N$8: track 0.00 -> 30.7 mm, vias 0 -> 1
- net N$28: track 0.00 -> 30.0 mm
- net N$7: track 0.00 -> 29.0 mm
- net N$11: track 0.00 -> 27.4 mm, vias 0 -> 1
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Other:
- board text added: "10"
- board text added: "11"
- board text added: "12"
- board text added: "13"
- board text added: "2"
- board text added: "3"
- board text added: "4"
- board text added: "5"
- board text added: "6"
- board text added: "7"
- board text added: "8"
- board text added: "9"
- board text added: "A0"
- board text added: "A1"
- board text added: "A2"
- board text added: "A3"
- board text added: "A4"
- board text added: "A5"
- board text added: "Arduino Pro Mini"
- board text added: "BLK"
- board text added: "GND"
- board text added: "GRN"
- board text added: "Keypad"
- board text added: "RAW"
- board text added: "RST"
- board text added: "RXI"
- board text added: "TXO"
- board text added: "VCC"

Commit message: production board REVA
Parts:
- JP6: device pinhead:1X02 -> pinhead:1X03
- moved JP4 1.91 mm to (26.7, 75.6)
- moved JP6 1.27 mm to (26.7, 68.6)
Connections:
- new net N$32: IC2.12, JP6.3
Routing:
- net N$4: track 19.2 -> 48.2 mm, vias 2 -> 0
- net N$27: track 18.5 -> 30.9 mm
- net N$15: track 40.8 -> 52.6 mm
- net N$32: track 0.00 -> 11.8 mm, vias 0 -> 1
- net N$19: track 33.4 -> 44.7 mm
- net N$3: track 40.8 -> 31.9 mm, vias 0 -> 1
- net N$8: track 30.7 -> 24.2 mm, vias 1 -> 2
- net N$14: track 43.1 -> 36.8 mm
- net N$16: track 36.8 -> 31.2 mm
- net GND: track 102.3 -> 97.4 mm, vias 2 -> 3
- net N$28: track 30.0 -> 25.9 mm
- net N$18: track 21.7 -> 25.7 mm
- net N$5: track 24.5 -> 27.8 mm, vias 1 -> 0
- net N$1: track 43.6 -> 46.2 mm, vias 0 -> 1
- net N$9: track 26.5 -> 24.6 mm
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